File: kukri.kicad_pcb (KiCad board)
At the start: 2 copper layers, 293 x 86.7 mm, 100 parts, among them SW1 SW_Push, U1 ProMicro

Commit message: added qmk support
Parts:
- added REF**: breakaway-mousebites, Keebio-Parts:breakaway-mousebites, F.Cu at (283.6, 112.6)
- added REF**: breakaway-mousebites, Keebio-Parts:breakaway-mousebites, F.Cu at (283.6, 106.5)
- added REF**: breakaway-mousebites, Keebio-Parts:breakaway-mousebites, F.Cu at (283.6, 99.1)
Routing:
- net c8: track 320.1 -> 323.3 mm
- net c7: track 376.4 -> 378.5 mm
- net GND: vias 3 -> 5
Other:
- outline, holes or cut-outs redrawn
